File: drone/hardware/kicad/Drone.kicad_pcb (KiCad board)
At the start: 2 copper layers, 94.6 x 94.6 mm, 119 parts, among them J1 USB_C_Receptacle_USB2.0, J2 Battery, J3 AE-VL53L0X, J4 B0067, J5 Motor1, J6 Motor2, J7 Motor3, J8 Motor4, Q1 SS8050-G, Q11 DMG3415U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

Commit message: ao
Parts:
- J6: value Motor2 -> Motor4
- J8: value Motor4 -> Motor2
Changed lines of the file:
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@@
       (effects (font (size 1 1) (thickness 0.15)))
     )
-    (fp_text value Motor2 (at 0 4.199999 315) (layer F.Fab)
+    (fp_text value Motor4 (at 0 4.199999 315) (layer F.Fab)
       (effects (font (size 1 1) (thickness 0.15)))
     )
@@
       (effects (font (size 1 1) (thickness 0.15)))
     )
-    (fp_text value Motor4 (at 0 4.199999 135) (layer F.Fab)
+    (fp_text value Motor2 (at 0 4.199999 135) (layer F.Fab)
       (effects (font (size 1 1) (thickness 0.15)))
     )
